File: singleboard/for.kicad_pcb (KiCad board)
At the start: 2 copper layers, 44 parts, among them P1 USB_OTG, P2 USB_OTG, U1 FT232RL, U2 STM32F103VETx, U3 MC33063/MC34063D_SO08, U4 AD620, U5 SKHMP*E010_SKHMPXE010, Y1 8MHz, Y2 32.768kHz

Commit message: PCB Progress
Parts:
- removed U3: MC33063/MC34063D_SO08, Housings_SOIC:SOIC-8_3.9x4.9mm_Pitch1.27mm
- removed U4: AD620, Housings_SOIC:SOIC-8_3.9x4.9mm_Pitch1.27mm
- added LED-COMMA1: LED, LEDs:LED_0805, F.Cu at (139.5, 106.6)
- added LED-COMMA2: LED, LEDs:LED_0805, F.Cu at (141.7, 106.6)
- added LED-COMMB1: LED, LEDs:LED_0805, F.Cu at (108.4, 104.5)
- added LED-COMMB2: LED, LEDs:LED_0805, F.Cu at (108.2, 107.4)
- added P-BT1: CONN_01X06, Pin_Headers:Pin_Header_Straight_1x06, B.Cu at (112.4, 114.6)
- added P-USB1: CONN_01X02, Pin_Headers:Pin_Header_Straight_1x02, B.Cu at (156.1, 116.8)
- added R-COMMA1: 330, Resistors_SMD:R_0805_HandSoldering, F.Cu at (139.4, 102.0)
- added R-COMMA2: 330, Resistors_SMD:R_0805_HandSoldering, F.Cu at (141.8, 102.0)
- added R-COMMB1: 330, Resistors_SMD:R_0805_HandSoldering, F.Cu at (103.6, 104.6)
- added R-COMMB2: 330, Resistors_SMD:R_0805_HandSoldering, F.Cu at (103.5, 107.3)
- added U-BATT1: MC33063/MC34063D_SO08, Housings_SOIC:SOIC-8_3.9x4.9mm_Pitch1.27mm, F.Cu at (86.9, 88.5)
- added U-SENSOR1: AD620, Housings_SOIC:SOIC-8_3.9x4.9mm_Pitch1.27mm, F.Cu at (104.4, 119.0)
- BATT-IN1, SW-LASER1, SW-PWR1: footprint Pin_Headers:Pin_Header_Straight_1x02 -> Connect:AK300-2; moved to B.Cu
- CP-PWR1, CP-PWR2, L-PWR1, P-BOOT1, P-PWR1, P-SENSOR1, P1, P2, U5, Y1, Y2: moved to B.Cu
- P-LASER1: value CONN_01X02 -> CONN_01X03; footprint Pin_Headers:Pin_Header_Straight_1x02 -> Pin_Headers:Pin_Header_Straight_1x03; moved to B.Cu
- moved P1 130.0 mm to (152.2, 129.3), turned to 90 degrees
- moved RV-PHLASER3 125.8 mm to (102.0, 125.5)
- moved R-PHLASER2 124.4 mm to (96.9, 118.2), turned to 180 degrees
- moved RV-PHLASER2 123.9 mm to (107.2, 125.5)
- moved P-SENSOR1 105.9 mm to (92.0, 123.5)
- moved R-PHLASER1 102.1 mm to (97.0, 120.5), turned to 180 degrees
- moved R-PHLASER3 94.4 mm to (97.0, 123.0)
- moved R-CLK1 90.9 mm to (108.0, 93.6), turned to 270 degrees
- moved RV-PHLASER1 90.5 mm to (104.2, 112.5), turned to 270 degrees
- moved C-PHLASER2 90.3 mm to (101.7, 129.8), turned to 180 degrees
- moved R-PWR2 88.0 mm to (89.0, 93.2), turned to 180 degrees
- moved SW-LASER1 79.0 mm to (72.2, 107.9), turned to 90 degrees
- moved P-LASER1 78.9 mm to (94.8, 102.3), turned to 180 degrees
- moved R-PWR3 77.8 mm to (83.3, 93.2), turned to 180 degrees
- moved C-PWR1 74.9 mm to (81.5, 88.3), turned to 90 degrees
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Connections:
- P1 pad 1: VCC -> Net-(P-USB1-Pad1)
- U2 pad 25: Net-(U2-Pad25) -> /BT_RX
- U2 pad 26: Net-(U2-Pad26) -> /BT_TX
Routing:
- net GND: track 0.00 -> 278.1 mm, vias 0 -> 3
- net VCC: track 0.00 -> 156.1 mm
- net VDD: track 0.00 -> 73.2 mm, vias 0 -> 4
- net Net-(CP-PWR2-Pad1): track 0.00 -> 64.6 mm, vias 0 -> 3
- net /ADC_SENSOR: track 0.00 -> 47.2 mm, vias 0 -> 2
- net /LCD_D0: track 0.00 -> 27.0 mm, vias 0 -> 1
- net /LCD_BL: track 0.00 -> 25.0 mm, vias 0 -> 1
- net /LCD_D1: track 0.00 -> 24.2 mm, vias 0 -> 1
- net Net-(C-CLK3-Pad1): track 0.00 -> 19.2 mm
- net Net-(C-CLK4-Pad1): track 0.00 -> 18.6 mm
- net Net-(D-PWR1-Pad2): track 0.00 -> 18.2 mm, vias 0 -> 1
- net Net-(C-PHLASER2-Pad2): track 0.00 -> 18.2 mm
- net Net-(CP-PWR1-Pad1): track 0.00 -> 17.6 mm, vias 0 -> 1
- net Net-(C-CLK1-Pad1): track 0.00 -> 17.5 mm
- net Net-(C-CLK2-Pad1): track 0.00 -> 17.4 mm
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
Commit message: PCB done
Parts:
- moved P-BOOT1 44.9 mm to (164.4, 63.8)
- moved C-CLK3 40.1 mm to (140.4, 72.7)
- moved C-CLK4 40.1 mm to (140.3, 75.0)
- moved P-PWR1 40.1 mm to (128.4, 53.9)
- moved P1 40.1 mm to (190.6, 117.8)
- moved U5 40.1 mm to (143.2, 66.7)
- moved R-COMMA2 40.1 mm to (180.3, 90.5)
- moved BATT-IN1 40.1 mm to (110.9, 67.5)
- moved CP-PWR2 40.1 mm to (130.5, 59.2)
- moved LED-COMMB1 40.1 mm to (146.9, 93.0)
- moved LED-COMMB2 40.1 mm to (146.7, 95.9)
- moved LED-PWR1 40.1 mm to (114.3, 83.6)
- moved R-COMMB1 40.1 mm to (142.1, 93.2)
- moved R-COMMB2 40.1 mm to (141.9, 95.8)
- moved R-LED1 40.1 mm to (109.5, 83.6)
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Routing:
- net VDD: track 73.2 -> 293.2 mm, vias 4 -> 19
- net GND: track 278.1 -> 493.1 mm, vias 3 -> 6
- net /TIN_INT: track 0.00 -> 110.9 mm, vias 0 -> 1
- net /LCD_D4: track 0.00 -> 106.9 mm, vias 0 -> 3
- net /LCD_D5: track 0.00 -> 106.8 mm, vias 0 -> 3
- net /TIN_CS: track 0.00 -> 101.5 mm, vias 0 -> 1
- net /LCD_CS: track 0.00 -> 100.9 mm, vias 0 -> 1
- net /LCD_D7: track 0.00 -> 98.4 mm, vias 0 -> 3
- net /LCD_D6: track 0.00 -> 98.2 mm, vias 0 -> 3
- net /LCD_D9: track 0.00 -> 91.9 mm, vias 0 -> 3
- net /LCD_D8: track 0.00 -> 91.9 mm, vias 0 -> 3
- net /TIN_MOSI: track 0.00 -> 90.5 mm, vias 0 -> 1
- net /LCD_D11: track 0.00 -> 86.4 mm, vias 0 -> 3
- net /LCD_D10: track 0.00 -> 86.0 mm, vias 0 -> 3
- net /TIN_MISO: track 0.00 -> 85.6 mm, vias 0 -> 3
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- added copper zone on B.Cu, net (none)
- added copper zone on F.Cu, net (none)
Other:
- board outline added: 121.4 x 75.7 mm
- net class Default: clearance 0.2 -> 0.1; via_dia 1.4 -> 1; via_drill 0.8 -> 0.6
- rule trace_clearance: 0.2 -> 0.1
- rule trace_min: 0.2 -> 0.05
