File: singleboard/for.sch (KiCad schematic (older format))
At the start: 44 parts, among them P1 USB_OTG, P2 USB_OTG, U1 FT232RL, U2 STM32F103VETx, U3 MC33063/MC34063D_SO08, U4 AD620, U5 SKHMP*E010_SKHMPXE010, Y1 8MHz, Y2 32.768kHz

Commit message: PCB Progress
Parts:
- removed P-LASER1: CONN_01X02, Pin_Headers:Pin_Header_Straight_1x02, symbol CONN_01X02
- added LED-COMMA1, LED-COMMA2, LED-COMMB1, LED-COMMB2: LED, LEDs:LED_0805, symbol LED
- added P-BT1: CONN_01X06, Pin_Headers:Pin_Header_Straight_1x06, symbol CONN_01X06
- added P-LASER1: CONN_01X03, Pin_Headers:Pin_Header_Straight_1x03, symbol CONN_01X03
- added P-USB1: CONN_01X02, Pin_Headers:Pin_Header_Straight_1x02, symbol CONN_01X02
- added R-COMMA1, R-COMMA2, R-COMMB1, R-COMMB2: 330, Resistors_SMD:R_0805_HandSoldering, symbol R
- BATT-IN1, SW-LASER1, SW-PWR1: footprint Pin_Headers:Pin_Header_Straight_1x02 -> Connect:AK300-2
- renumbered U3 to U-BATT1, U4 to U-SENSOR1
Connections:
- net GND: now also P-BT1.3 (P3), P-LASER1.2 (P2), P-LASER1.3 (P3)
- net RX: now also LED-COMMA1.1 (K)
- net TX: now also LED-COMMA2.1 (K)
- net VCC: now also P-USB1.2 (P2); no longer P1.1 (VBUS)
- net VDD: now also P-BT1.2 (P2), R-COMMA1.1, R-COMMA2.1, R-COMMB1.1, R-COMMB2.1
- net BT_RX: now reaches U2.25 (ADC1_IN2/ADC2_IN2/ADC3_IN2/TIM2_CH3/TIM5_CH3/USART2_TX/PA2)
- net BT_RX: now also LED-COMMB1.1 (K), P-BT1.5 (P5)
- net BT_TX: now reaches U2.26 (ADC1_IN3/ADC2_IN3/ADC3_IN3/TIM2_CH4/TIM5_CH4/USART2_RX/PA3)
- net BT_TX: now also LED-COMMB2.1 (K), P-BT1.4 (P4)
- net at D-LASER1.1 (K), D-LASER2.1 (K): now also P-LASER1.1 (P1)
- new net: LED-COMMA1.2 (A), R-COMMA1.2
- new net: LED-COMMA2.2 (A), R-COMMA2.2
- new net: LED-COMMB1.2 (A), R-COMMB1.2
- new net: LED-COMMB2.2 (A), R-COMMB2.2
- new net: P-USB1.1 (P1), P1.1 (VBUS)
