File: Model_3D/pcb/pcb_usb/for_usb.kicad_pcb (KiCad board)
At the start: 2 copper layers, 121.4 x 75.7 mm, 54 parts, among them P1 USB_OTG, P2 USB_OTG, U1 FT232RL, U2 STM32F103VETx, U5 SKHMP*E010_SKHMPXE010, Y1 8MHz, Y2 32.768kHz

Commit message: model 3d
Parts:
- added G***: LOGO, logo_lab:logo, B.Cu at (165.5, 85.4)
