File: opm_addon/opm.kicad_pcb (KiCad board)
At the start: 2 copper layers, 27 parts, among them U1 AD620, U2 AD620

Commit message: opm
Parts:
- removed 100K1, 100K2: POT_TRIM, Potentiometers:Potentiometer_Trimmer-EVM3E
- added RV-LOOP1: 100K, Potentiometers:Potentiometer_Trimmer-EVM3E, F.Cu at (103.4, 104.3)
- added RV-LOOP2: 100K, Potentiometers:Potentiometer_Trimmer-EVM3E, F.Cu at (103.9, 82.1)
- P-IN1, P-IN2, P-LASER1, P-PIN1, SW-PWR1: moved to B.Cu
- moved C-LOOP1 79.5 mm to (107.1, 104.5), turned to 270 degrees
- moved RV-REF1 76.5 mm to (112.8, 97.7), turned to 90 degrees
- moved RV-REF2 72.1 mm to (113.3, 75.2), turned to 90 degrees
- moved U1 71.9 mm to (103.2, 97.9)
- moved RV-GAIN1 70.3 mm to (103.1, 92.1)
- moved SW-PWR1 63.7 mm to (113.2, 54.7), turned to 270 degrees
- moved C-REF1 58.1 mm to (116.9, 97.8), turned to 270 degrees
- moved R-LED1 56.7 mm to (103.2, 51.3)
- moved U2 55.3 mm to (103.7, 75.6)
- moved R-INPLUS1 54.6 mm to (95.0, 99.0), turned to 180 degrees
- moved C-REF2 53.9 mm to (117.4, 75.0), turned to 270 degrees
- moved R-INMIN2 52.3 mm to (96.2, 74.5), turned to 180 degrees
- moved P-PIN1 46.7 mm to (125.2, 52.4), turned to 180 degrees
- moved R-IN-PLUS1 43.8 mm to (95.0, 101.4)
- moved LED1 43.6 mm to (98.4, 51.3)
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Connections:
- P-PIN1 pad 1: GND -> /PIN_VDD
- P-PIN1 pad 10: /ADC1 -> /ADC0
- P-PIN1 pad 2: /PIN_VDD -> GND
- P-PIN1 pad 45: Net-(P-PIN1-Pad45) -> /PIN_VCC
- P-PIN1 pad 46: Net-(P-PIN1-Pad46) -> GND
- P-PIN1 pad 9: /ADC0 -> /ADC1
Routing:
- net GND: track 0.00 -> 192.8 mm
- net /PIN_VCC: track 0.00 -> 131.9 mm, vias 0 -> 4
- net /ADC1: track 0.00 -> 86.9 mm, vias 0 -> 2
- net VCC: track 0.00 -> 77.3 mm
- net /ADC0: track 0.00 -> 36.5 mm, vias 0 -> 2
- net /PIN_VDD: track 0.00 -> 20.8 mm
- net Net-(C-LOOP1-Pad2): track 0.00 -> 19.1 mm
- net Net-(C-LOOP2-Pad2): track 0.00 -> 18.1 mm
- net Net-(D-LASER1-Pad1): track 0.00 -> 10.3 mm
- net Net-(D-LASER1-Pad2): track 0.00 -> 9.25 mm
- net Net-(RV-GAIN2-Pad2): track 0.00 -> 9.22 mm
- net Net-(R-IN-PLUS1-Pad1): track 0.00 -> 7.99 mm
- net Net-(R-IN-PLUS2-Pad1): track 0.00 -> 7.56 mm
- net Net-(RV-GAIN1-Pad2): track 0.00 -> 7.51 mm
- net Net-(RV-REF2-Pad2): track 0.00 -> 6.28 mm
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Other:
- board outline added: 44.1 x 68.2 mm
- net class Default: via_dia 0.6 -> 1.6; via_drill 0.4 -> 0.8
