File: opm_addon/opm.sch (KiCad schematic (older format))
At the start: 25 parts, among them U1 AD620, U2 AD620

Commit message: opm
Parts:
- added LED1: LED, LEDs:LED_0805, symbol LED
- added R-LED1: 330, Resistors_SMD:R_0805_HandSoldering, symbol R
- 100K1, 100K2, RV-GAIN1, RV-GAIN2, RV-REF1, RV-REF2: footprint (none) -> Potentiometers:Potentiometer_Trimmer-EVM3E
- C-LOOP1, C-LOOP2, C-REF1, C-REF2: footprint (none) -> Capacitors_SMD:C_0805_HandSoldering
- D-LASER1: footprint (none) -> Diodes_SMD:MELF_Handsoldering
- D-LASER2: footprint (none) -> Diodes_SMD:SMB_Handsoldering
- P-IN1, P-IN2, P-LASER1: footprint (none) -> Pin_Headers:Pin_Header_Straight_1x03
- P-PIN1: renamed from P-PIN; footprint (none) -> Pin_Headers:Pin_Header_Straight_2x23
- R-IN-PLUS1, R-IN-PLUS2, R-INMIN1, R-INMIN2, R-INPLUS1, R-INPLUS2: footprint (none) -> Resistors_SMD:R_0805_HandSoldering
- SW-PWR1: footprint (none) -> switch-dil:DIP02YL
- U1, U2: footprint (none) -> Housings_SOIC:SOIC-8_3.9x4.9mm_Pitch1.27mm
Connections:
- net GND: now also LED1.1 (K)
- net PIN_VDD: now also P-PIN1.7 (P7), P-PIN1.8 (P8)
- net VCC: now also R-LED1.2
- new net: LED1.2 (A), R-LED1.1

Commit message: opm
Parts:
- RV-LOOP1: renamed from 100K1; value POT_TRIM -> 100K
- RV-LOOP2: renamed from 100K2; value POT_TRIM -> 100K
Connections:
- net ADC0: now also P-PIN1.10 (P10); no longer P-PIN1.9 (P9)
- net ADC1: now also P-PIN1.9 (P9); no longer P-PIN1.10 (P10)
- net GND: now also P-PIN1.2 (P2), P-PIN1.46 (P46); no longer P-PIN1.1 (P1)
- net PIN_VCC: now also P-PIN1.45 (P45)
- net PIN_VDD: now also P-PIN1.1 (P1); no longer P-PIN1.2 (P2)
Changed lines of the file:
@@
 $EndComp
 $Comp
-L POT_TRIM 100K2
+L POT_TRIM RV-LOOP2
 U 1 1 58BE54E9
 P 2700 3100
-F 0 "100K2" V 2525 3100 50  0000 C CNN
-F 1 "POT_TRIM" V 2600 3100 50  0000 C CNN
+F 0 "RV-LOOP2" V 2525 3100 50  0000 C CNN
+F 1 "100K" V 2600 3100 50  0000 C CNN
 F 2 "Potentiometers:Potentiometer_Trimmer-EVM3E" H 2700 3100 50  0001 C CNN
 F 3 "" H 2700 3100 50  0000 C CNN
@@
 $EndComp
 $Comp
-L POT_TRIM 100K1
+L POT_TRIM RV-LOOP1
 U 1 1 58BE762B
 P 2600 5650
-F 0 "100K1" V 2425 5650 50  0000 C CNN
-F 1 "POT_TRIM" V 2500 5650 50  0000 C CNN
+F 0 "RV-LOOP1" V 2425 5650 50  0000 C CNN
+F 1 "100K" V 2500 5650 50  0000 C CNN
 F 2 "Potentiometers:Potentiometer_Trimmer-EVM3E" H 2600 5650 50  0001 C CNN
 F 3 "" H 2600 5650 50  0000 C CNN
@@
 F 3 "" H 5050 3650 50  0000 C CNN
 	1    5050 4500
-	1    0    0    -1
+	-1   0    0    -1
 $EndComp
 $Comp
@@
 	1    0    0    -1
 $EndComp
-Text Label 5550 3400 0    60   ~ 0
-PIN_VDD
 Text Label 3650 2250 0    60   ~ 0
 ADC0
 Text Label 3550 4800 0    60   ~ 0
-ADC1
-Text Label 4600 3800 0    60   ~ 0
-ADC0
-Text Label 5500 3800 0    60   ~ 0
 ADC1
 $Comp
@@
 	3400 2250 3400 3300
 Wire Wire Line
-	2700 2950 2700 2350
+	2700 2350 2700 2950
 Wire Wire Line
 	2250 2350 2250 2400
@@
 	3300 4800 3300 5850
 Wire Wire Line
-	2600 5500 2600 4900
+	2600 4900 2600 5500
 Wire Wire Line
 	2150 4900 2150 4950
@@
 	5050 1700 4900 1700
 Wire Wire Line
+	3400 2250 3650 2250
+Wire Wire Line
+	3300 4800 3550 4800
+Wire Wire Line
+	4950 2600 4850 2600
+Wire Wire Line
+	4450 2600 4550 2600
+Wire Wire Line
+	4150 2600 4050 2600
+Wire Wire Line
 	4800 3400 4500 3400
 Wire Wire Line
-	5300 3400 5550 3400
-Wire Wire Line
-	4800 3700 5400 3700
-Wire Wire Line
-	3400 2250 3650 2250
-Wire Wire Line
-	3300 4800 3550 4800
-Wire Wire Line
-	4800 3800 4600 3800
+	5300 3400 5500 3400
+Text Label 5500 3400 0    60   ~ 0
+PIN_VDD
+Wire Wire Line
+	4800 3700 4500 3700
+Text Label 4500 3700 0    60   ~ 0
+PIN_VDD
+Wire Wire Line
+	5300 3700 5500 3700
+Text Label 5500 3700 0    60   ~ 0
+PIN_VDD
+Wire Wire Line
+	4800 3800 4500 3800
+Text Label 4500 3800 0    60   ~ 0
+ADC0
 Wire Wire Line
 	5300 3800 5500 3800
-Wire Wire Line
-	4950 2600 4850 2600
-Wire Wire Line
-	4450 2600 4550 2600
-Wire Wire Line
-	4150 2600 4050 2600
-Wire Wire Line
-	5400 3700 5400 3400
-Connection ~ 5400 3400
-Connection ~ 5300 3700
+Text Label 5500 3800 0    60   ~ 0
+ADC1
+$Comp
+L GND #PWR?
+U 1 1 58BF3840
+P 4500 5600
+F 0 "#PWR?" H 4500 5350 50  0001 C CNN
+F 1 "GND" H 4500 5450 50  0000 C CNN
+F 2 "" H 4500 5600 50  0000 C CNN
+F 3 "" H 4500 5600 50  0000 C CNN
+	1    4500 5600
+	1    0    0    -1
+$EndComp
+Wire Wire Line
+	4800 5600 4500 5600
+Wire Wire Line
+	5300 5600 5500 5600
+Text Label 5500 5600 0    60   ~ 0
+PIN_VCC
 $EndSCHEMATC
