File: new_pcb/new_pcb.kicad_pcb (KiCad board)
At the start: 2 copper layers, 73 parts, among them P1 USB_OTG, P2 USB_OTG, U1 STM32F407VGTx, U2 H28, U3 FT232RL, U4 LM317_SOT223, Y1 24MHz, Y2 32kHz

Commit message: progress
Parts:
- added D-BATT1: D, Diodes_SMD:D_SMB_Standard, F.Cu at (246.2, 72.3)
- U3: footprint Housings_SSOP:TSSOP-28_4.4x9.7mm_Pitch0.65mm -> Housings_SSOP:SSOP-28_5.3x10.2mm_Pitch0.65mm
- moved R-TX1 5.15 mm to (203.8, 86.4)
- moved R-RX1 5.13 mm to (206.1, 86.5)
- moved U3 0.77 mm to (207.7, 73.8)
Connections:
- P2 pad 1: Net-(BATT-IN1-Pad1) -> Net-(D-BATT1-Pad2)
Routing:
- net VDD: track 506.0 -> 540.9 mm
- net GND: track 736.0 -> 763.5 mm
- net Net-(BATT-IN1-Pad1): track 38.7 -> 28.8 mm
- net Net-(D-BATT1-Pad2): track 0.00 -> 5.67 mm
- net /TX: track 76.5 -> 71.4 mm
- net /RX: track 81.5 -> 76.5 mm
- net VCC: track 537.8 -> 542.1 mm
- net Net-(R-TX1-Pad2): track 3.57 -> 7.79 mm
- net Net-(R-RX1-Pad2): track 3.83 -> 7.72 mm
- net Net-(P1-Pad3): track 10.3 -> 8.76 mm
- net Net-(P1-Pad2): track 14.0 -> 12.9 mm
