File: new_pcb/new_pcb.sch (KiCad schematic (older format))
At the start: 73 parts, among them P1 USB_OTG, P2 USB_OTG, U1 STM32F407VGTx, U2 H28, U3 FT232RL, U4 LM317_SOT223, Y1 24MHz, Y2 32kHz

Commit message: new design
Connections:
- net GLCD_RS: now also U1.78 (DCMI_D8/I2S3_CK/SDIO_D2/SPI3_SCK/UART4_TX/USART3_TX/PC10); no longer U1.80 (DCMI_D9/I2S3_SD/SDIO_CK/SPI3_MOSI/UART5_TX/USART3_CK/PC12)
- net GLCD_RST: now also U1.80 (DCMI_D9/I2S3_SD/SDIO_CK/SPI3_MOSI/UART5_TX/USART3_CK/PC12); no longer U1.78 (DCMI_D8/I2S3_CK/SDIO_D2/SPI3_SCK/UART4_TX/USART3_TX/PC10)
Changed lines of the file:
@@
 GLCD_CS2
 Text Label 16650 9550 0    60   ~ 0
-GLCD_RST
+GLCD_RS
 Text Label 15800 2900 1    60   ~ 0
 GLCD_RST
@@
 GLCD_RW
 Text Label 16650 9750 0    60   ~ 0
-GLCD_RS
+GLCD_RST
 Text Label 16000 2900 1    60   ~ 0
 GLCD_RS

Commit message: progress
Parts:
- added D-BATT1: D, Diodes_SMD:D_SMB_Standard, symbol D
- U3: footprint Housings_SSOP:TSSOP-28_4.4x9.7mm_Pitch0.65mm -> Housings_SSOP:SSOP-28_5.3x10.2mm_Pitch0.65mm
Connections:
- net at BATT-IN1.1 (P1), P-PWR2.2 (P2): now also D-BATT1.1 (K); no longer P2.1 (VBUS)
- new net: D-BATT1.2 (A), P2.1 (VBUS)
