File: new_pcb/sub-design/core/new_pcb.kicad_pcb (KiCad board)
At the start: 2 copper layers, 52.5 x 46.8 mm, 3 parts, among them U1 STM32F407VGTx

Commit message: progress
Parts:
- J-CPU1, J-CPU2: moved to B.Cu
- turned J-CPU1 to 180 degrees
- turned J-CPU2 to 0 degrees
Other:
- board size 52.5 x 46.8 mm -> 54.5 x 46.9 mm

Commit message: progres hardware oke
Routing:
- net VDD: track 218.8 -> 155.6 mm, vias 2 -> 9
- net GND: track 109.4 -> 132.3 mm
- net /BOOT: track 35.6 -> 41.0 mm
- net /ADC_SCL: track 32.6 -> 36.9 mm
- net /ADC_SDA: track 34.3 -> 38.2 mm
- net /ADC_EOC: track 31.2 -> 34.4 mm
- net /GLCD_RST: track 25.3 -> 27.2 mm
- net /USER_INPUT_2: track 32.3 -> 31.0 mm
- net /ADC_XCLR: track 30.3 -> 31.7 mm
- net /ADC_MCLK: track 28.9 -> 30.2 mm
- net /GLCD_RW: track 25.4 -> 26.5 mm
- net /RST: track 21.9 -> 21.0 mm
- net /OSC24_IN: track 23.8 -> 23.0 mm
- net /GLCD_CS1: track 21.7 -> 21.0 mm
- net /OSC24_OUT: track 22.9 -> 22.2 mm
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Other:
- board size 54.5 x 46.9 mm -> 51.3 x 45 mm
