File: circuit/pwr_dist/pwr_dist.kicad_pcb (KiCad board)
At the start: 2 copper layers, 34.3 x 43.8 mm, 5 parts, among them J1 CONN_01X02, J2 CONN_01X02, J3 CONN_01X02

Commit message: last progress
Parts:
- added REF**: MountingHole_2.5mm, Mounting_Holes:MountingHole_2.5mm, F.Cu at (88.0, 71.7)
- added REF**: MountingHole_2.5mm, Mounting_Holes:MountingHole_2.5mm, F.Cu at (88.0, 54.8)
- added REF**: MountingHole_2.5mm, Mounting_Holes:MountingHole_2.5mm, F.Cu at (113.8, 36.8)
Changed lines of the file:
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@@
     (links 9)
     (no_connects 0)
-    (area 76.649999 32.769999 117.725001 77.085001)
+    (area 76.649999 32.375 121.878572 77.085001)
     (thickness 1.6)
     (drawings 4)
     (tracks 28)
     (zones 0)
-    (modules 5)
+    (modules 8)
     (nets 6)
   )
@@
     (visible_elements FFFFEF7F)
     (pcbplotparams
-      (layerselection 0x00030_80000001)
+      (layerselection 0x00000_00000001)
       (usegerberextensions false)
-      (excludeedgelayer true)
+      (excludeedgelayer false)
       (linewidth 0.100000)
       (plotframeref false)
-      (viasonmask false)
+      (viasonmask true)
       (mode 1)
       (useauxorigin false)
@@
       (outputformat 4)
       (mirror false)
-      (drillshape 0)
+      (drillshape 2)
       (scaleselection 1)
       (outputdirectory ""))
@@
     )
   )
+  (module Mounting_Holes:MountingHole_2.5mm (layer F.Cu)
+    (at 88 71.7)
+    (descr "Mounting Hole 2.5mm, no annular")
+    (tags "mounting hole 2.5mm no annular")
+    (fp_text reference REF** (at 0 -3.5) (layer F.SilkS)
+      (effects (font (size 1 1) (thickness 0.15)))
+    )
+    (fp_text value MountingHole_2.5mm (at 0 3.5) (layer F.Fab)
+      (effects (font (size 1 1) (thickness 0.15)))
+    )
+    (fp_circle (center 0 0) (end 2.5 0) (layer Cmts.User) (width 0.15))
+    (fp_circle (center 0 0) (end 2.75 0) (layer F.CrtYd) (width 0.05))
+    (pad 1 np_thru_hole circle (at 0 0) (size 2.5 2.5) (drill 2.5) (layers *.Cu *.Mask))
+  )
+  (module Mounting_Holes:MountingHole_2.5mm (layer F.Cu)
+    (at 88 54.8)
+    (descr "Mounting Hole 2.5mm, no annular")
+    (tags "mounting hole 2.5mm no annular")
+    (fp_text reference REF** (at 0 -3.5) (layer F.SilkS)
+      (effects (font (size 1 1) (thickness 0.15)))
+    )
+    (fp_text value MountingHole_2.5mm (at 0 3.5) (layer F.Fab)
+      (effects (font (size 1 1) (thickness 0.15)))
+    )
+    (fp_circle (center 0 0) (end 2.5 0) (layer Cmts.User) (width 0.15))
+    (fp_circle (center 0 0) (end 2.75 0) (layer F.CrtYd) (width 0.05))
+    (pad 1 np_thru_hole circle (at 0 0) (size 2.5 2.5) (drill 2.5) (layers *.Cu *.Mask))
+  )
+  (module Mounting_Holes:MountingHole_2.5mm (layer F.Cu)
+    (at 113.8 36.8)
+    (descr "Mounting Hole 2.5mm, no annular")
+    (tags "mounting hole 2.5mm no annular")
+    (fp_text reference REF** (at 0 -3.5) (layer F.SilkS)
+      (effects (font (size 1 1) (thickness 0.15)))
+    )
+    (fp_text value MountingHole_2.5mm (at 0 3.5) (layer F.Fab)
+      (effects (font (size 1 1) (thickness 0.15)))
+    )
+    (fp_circle (center 0 0) (end 2.5 0) (layer Cmts.User) (width 0.15))
+    (fp_circle (center 0 0) (end 2.75 0) (layer F.CrtYd) (width 0.05))
+    (pad 1 np_thru_hole circle (at 0 0) (size 2.5 2.5) (drill 2.5) (layers *.Cu *.Mask))
+  )
   (gr_line (start 83.185 76.835) (end 83.185 33.02) (layer Edge.Cuts) (width 0.5))
